File: kicad_project_files/keych&chong/keych&chong.kicad_sch (KiCad schematic)
At the start: 233 parts, among them J1 USB_C_Receptacle_USB2.0, U1 ATmega32U4-A, Y1 16mhz

Commit message: remove diode
Parts:
- removed D?: 1N4148, Diode_THT:D_DO-35_SOD27_P7.62mm_Horizontal, symbol Diode:1N4148
Connections:
- net VCC: now also J1.A4 (VBUS), J1.A9 (VBUS), J1.B4 (VBUS), J1.B9 (VBUS)
Changed lines of the file:
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@@
   (junction (at 208.28 85.09) (diameter 0) (color 0 0 0 0)
   )
+  (junction (at 370.84 173.99) (diameter 0) (color 0 0 0 0)
+  )
   (junction (at 76.2 161.29) (diameter 0) (color 0 0 0 0)
   )
@@
   (junction (at 76.2 139.7) (diameter 0) (color 0 0 0 0)
   )
-  (junction (at 378.46 173.99) (diameter 0) (color 0 0 0 0)
-  )
   (junction (at 55.88 63.5) (diameter 0) (color 0 0 0 0)
   )
@@
     (stroke (width 0) (type default) (color 0 0 0 0))
   )
-  (wire (pts (xy 378.46 173.99) (xy 383.54 173.99))
+  (wire (pts (xy 370.84 173.99) (xy 375.92 173.99))
     (stroke (width 0) (type default) (color 0 0 0 0))
   )
@@
     (stroke (width 0) (type default) (color 0 0 0 0))
   )
-  (wire (pts (xy 378.46 167.64) (xy 378.46 173.99))
+  (wire (pts (xy 370.84 167.64) (xy 370.84 173.99))
     (stroke (width 0) (type default) (color 0 0 0 0))
   )
@@
     (pin "4")
   )
-  (symbol (lib_id "power:PWR_FLAG") (at 378.46 167.64 0) (unit 1)
+  (symbol (lib_id "power:PWR_FLAG") (at 370.84 167.64 0) (unit 1)
     (in_bom yes) (on_board yes) (fields_autoplaced)
-    (property "Reference" "#FLG?" (id 0) (at 378.46 165.735 0)
+    (property "Reference" "#FLG?" (id 0) (at 370.84 165.735 0)
       (effects (font (size 1.27 1.27)) hide)
     )
-    (property "Value" "PWR_FLAG" (id 1) (at 378.46 162.56 0))
-    (property "Footprint" "" (id 2) (at 378.46 167.64 0)
+    (property "Value" "PWR_FLAG" (id 1) (at 370.84 162.56 0))
+    (property "Footprint" "" (id 2) (at 370.84 167.64 0)
       (effects (font (size 1.27 1.27)) hide)
     )
-    (property "Datasheet" "~" (id 3) (at 378.46 167.64 0)
+    (property "Datasheet" "~" (id 3) (at 370.84 167.64 0)
       (effects (font (size 1.27 1.27)) hide)
     )
@@
     (pin "2")
   )
-  (symbol (lib_id "Diode:1N4148") (at 374.65 173.99 180) (unit 1)
-    (in_bom yes) (on_board yes) (fields_autoplaced)
-    (property "Reference" "D?" (id 0) (at 374.65 167.64 0))
-    (property "Value" "1N4148" (id 1) (at 374.65 170.18 0))
-    (property "Footprint" "Diode_THT:D_DO-35_SOD27_P7.62mm_Horizontal" (id 2) (at 374.65 169.545 0)
-      (effects (font (size 1.27 1.27)) hide)
-    )
-    (property "Datasheet" "https://assets.nexperia.com/documents/data-sheet/1N4148_1N4448.pdf" (id 3) (at 374.65 173.99 0)
-      (effects (font (size 1.27 1.27)) hide)
-    )
-    (pin "1")
-    (pin "2")
-  )
   (symbol (lib_id "Diode:1N4148") (at 213.36 157.48 90) (unit 1)
     (in_bom yes) (on_board yes) (fields_autoplaced)
@@
     (pin "4")
   )
-  (symbol (lib_id "power:VCC") (at 383.54 173.99 0) (unit 1)
+  (symbol (lib_id "power:VCC") (at 375.92 173.99 0) (unit 1)
     (in_bom yes) (on_board yes) (fields_autoplaced)
-    (property "Reference" "#PWR09" (id 0) (at 383.54 177.8 0)
+    (property "Reference" "#PWR09" (id 0) (at 375.92 177.8 0)
       (effects (font (size 1.27 1.27)) hide)
     )
-    (property "Value" "VCC" (id 1) (at 383.54 168.91 0))
-    (property "Footprint" "" (id 2) (at 383.54 173.99 0)
+    (property "Value" "VCC" (id 1) (at 375.92 168.91 0))
+    (property "Footprint" "" (id 2) (at 375.92 173.99 0)
       (effects (font (size 1.27 1.27)) hide)
     )
-    (property "Datasheet" "" (id 3) (at 383.54 173.99 0)
+    (property "Datasheet" "" (id 3) (at 375.92 173.99 0)
       (effects (font (size 1.27 1.27)) hide)
     )
@@
       (reference "D106") (unit 1) (value "LED") (footprint "")
     )
-    (path "/1767b76a-d6ac-48b3-a8f6-ed12f684902a"
-      (reference "D?") (unit 1) (value "1N4148") (footprint "Diode_THT:D_DO-35_SOD27_P7.62mm_Horizontal")
-    )
     (path "/fab12cff-f0ef-4023-9d9a-1274eae4f0d8"

Commit message: add footprints
Parts:
- C1, C2, C3, C4, C5, C6, C8: footprint (none) -> Capacitor_SMD:C_1206_3216Metric_Pad1.33x1.80mm_HandSolder
- C7: value 1µF -> 1uf; footprint (none) -> Capacitor_SMD:C_1206_3216Metric_Pad1.33x1.80mm_HandSolder; symbol Device:C_Polarized -> Device:C
- D1, D10, D100, D101, D102, D103, D104, D11, D12, D13, D14, D15, D16, D17, D18, D19, D2, D20, D21, D22, D23, D24, D25, D26, D27, D28, D29, D3, D30, D31, D32, D33, D34, D35, D36, D37, D38, D39, D4, D40, D41, D42, D43, D44, D45, D46, D47, D48, D49, D5, D50, D51, D52, D53, D54, D55, D56, D57, D58, D59, D6, D60, D61, D62, D63, D64, D65, D66, D67, D68, D69, D7, D70, D71, D72, D73, D74, D75, D76, D77, D78, D79, D8, D80, D81, D82, D83, D84, D85, D86, D87, D88, D89, D9, D90, D91, D92, D93, D94, D95, D96, D97, D98, D99: footprint Diode_THT:D_DO-35_SOD27_P7.62mm_Horizontal -> Diode_SMD:D_SOD-123
- SW_0, SW_1, SW_2, SW_3, SW_4, SW_5, SW_6, SW_7, SW_8, SW_9, SW_A1, SW_ALT1, SW_B1, SW_BACKSPACE1, SW_BK-SLH1, SW_C1, SW_CAPS1, SW_CLO-BRC1, SW_CLS-BRC1, SW_COLON1, SW_D1, SW_DASH1, SW_DELETE1, SW_DOWN1, SW_E1, SW_END1, SW_ENT1, SW_ESC1, SW_F1, SW_F10, SW_F11, SW_F12, SW_F13, SW_F2, SW_F3, SW_F4, SW_F5, SW_F6, SW_F7, SW_F8, SW_F9, SW_FN1, SW_G1, SW_H1, SW_HOME1, SW_I1, SW_INSERT1, SW_J1, SW_K1, SW_L-ALT1, SW_L-CTRL1, SW_L-SHFT1, SW_L1, SW_LEFT1, SW_M1, SW_MENU1, SW_N1, SW_NUM-ASTR1, SW_NUM-DEL1, SW_NUM-ENT1, SW_NUM-FWD-SLH1, SW_NUM-LK1, SW_NUM-MINUS1, SW_NUM-PLUS1, SW_NUM0, SW_NUM1, SW_NUM2, SW_NUM3, SW_NUM4, SW_NUM5, SW_NUM6, SW_NUM7, SW_NUM8, SW_NUM9, SW_O1, SW_OPN-BRC1, SW_OPN-BRC2, SW_P1, SW_PG-DN1, SW_PG-UP1, SW_PLUS1, SW_PRT-SC1, SW_PSE-BK1, SW_Q1, SW_QSTN1, SW_QUOTE1, SW_R-CTRL1, SW_R-SHFT1, SW_R1, SW_RIGHT1, SW_S1, SW_SCRL-LK1, SW_SPACE1, SW_T1, SW_TAB1, SW_TILDA1, SW_U1, SW_UP1, SW_V1, SW_W1, SW_WIN1, SW_X1, SW_Y1, SW_Z1: value SW_MEC_5G -> SW_SPST; symbol Switch:SW_MEC_5G -> Switch:SW_SPST
- SW_RESET1: renamed from SW_RESET; value SW_MEC_5G -> SW_SPST; symbol Switch:SW_MEC_5G -> Switch:SW_SPST
- gave numbers to parts that had none: 1
- renumbered ISCP to ISCP1
Connections:
- net COL_1: now also SW_CAPS1.2 (B), SW_F12.2 (B), SW_INSERT1.2 (B), SW_L-CTRL1.2 (B), SW_L-SHFT1.2 (B), SW_TAB1.2 (B), SW_TILDA1.2 (B); no longer SW_CAPS1.3 (B), SW_CAPS1.4 (B), SW_F12.3 (B), SW_F12.4 (B), SW_INSERT1.3 (B), SW_INSERT1.4 (B), SW_L-CTRL1.3 (B), SW_L-CTRL1.4 (B), SW_L-SHFT1.3 (B), SW_L-SHFT1.4 (B), SW_TAB1.3 (B), SW_TAB1.4 (B), SW_TILDA1.3 (B), SW_TILDA1.4 (B)
- net COL_10: now also SW_9.2 (B), SW_CLS-BRC1.2 (B), SW_F8.2 (B), SW_L1.2 (B), SW_NUM-DEL1.2 (B), SW_O1.2 (B); no longer SW_9.3 (B), SW_9.4 (B), SW_CLS-BRC1.3 (B), SW_CLS-BRC1.4 (B), SW_F8.3 (B), SW_F8.4 (B), SW_L1.3 (B), SW_L1.4 (B), SW_NUM-DEL1.3 (B), SW_NUM-DEL1.4 (B), SW_O1.3 (B), SW_O1.4 (B)
- net COL_11: now also SW_0.2 (B), SW_COLON1.2 (B), SW_HOME1.2 (B), SW_NUM1.2 (B), SW_P1.2 (B), SW_QSTN1.2 (B); no longer SW_0.3 (B), SW_0.4 (B), SW_COLON1.3 (B), SW_COLON1.4 (B), SW_HOME1.3 (B), SW_HOME1.4 (B), SW_NUM1.3 (B), SW_NUM1.4 (B), SW_P1.3 (B), SW_P1.4 (B), SW_QSTN1.3 (B), SW_QSTN1.4 (B)
- net COL_12: now also SW_DASH1.2 (B), SW_END1.2 (B), SW_NUM2.2 (B), SW_OPN-BRC2.2 (B), SW_QUOTE1.2 (B), SW_R-SHFT1.2 (B); no longer SW_DASH1.3 (B), SW_DASH1.4 (B), SW_END1.3 (B), SW_END1.4 (B), SW_NUM2.3 (B), SW_NUM2.4 (B), SW_OPN-BRC2.3 (B), SW_OPN-BRC2.4 (B), SW_QUOTE1.3 (B), SW_QUOTE1.4 (B), SW_R-SHFT1.3 (B), SW_R-SHFT1.4 (B)
- net COL_13: now also SW_CLO-BRC1.2 (B), SW_DELETE1.2 (B), SW_ENT1.2 (B), SW_LEFT1.2 (B), SW_NUM3.2 (B), SW_PLUS1.2 (B); no longer SW_CLO-BRC1.3 (B), SW_CLO-BRC1.4 (B), SW_DELETE1.3 (B), SW_DELETE1.4 (B), SW_ENT1.3 (B), SW_ENT1.4 (B), SW_LEFT1.3 (B), SW_LEFT1.4 (B), SW_NUM3.3 (B), SW_NUM3.4 (B), SW_PLUS1.3 (B), SW_PLUS1.4 (B)
- net COL_14: now also SW_BACKSPACE1.2 (B), SW_BK-SLH1.2 (B), SW_DOWN1.2 (B), SW_F9.2 (B), SW_NUM4.2 (B), SW_UP1.2 (B); no longer SW_BACKSPACE1.3 (B), SW_BACKSPACE1.4 (B), SW_BK-SLH1.3 (B), SW_BK-SLH1.4 (B), SW_DOWN1.3 (B), SW_DOWN1.4 (B), SW_F9.3 (B), SW_F9.4 (B), SW_NUM4.3 (B), SW_NUM4.4 (B), SW_UP1.3 (B), SW_UP1.4 (B)
- net COL_15: now also SW_F10.2 (B), SW_NUM5.2 (B), SW_NUM7.2 (B), SW_NUM8.2 (B), SW_PRT-SC1.2 (B), SW_RIGHT1.2 (B); no longer SW_F10.3 (B), SW_F10.4 (B), SW_NUM5.3 (B), SW_NUM5.4 (B), SW_NUM7.3 (B), SW_NUM7.4 (B), SW_NUM8.3 (B), SW_NUM8.4 (B), SW_PRT-SC1.3 (B), SW_PRT-SC1.4 (B), SW_RIGHT1.3 (B), SW_RIGHT1.4 (B)
- net COL_16: now also SW_F11.2 (B), SW_NUM-ENT1.2 (B), SW_NUM-FWD-SLH1.2 (B), SW_NUM6.2 (B), SW_NUM9.2 (B), SW_SCRL-LK1.2 (B); no longer SW_F11.3 (B), SW_F11.4 (B), SW_NUM-ENT1.3 (B), SW_NUM-ENT1.4 (B), SW_NUM-FWD-SLH1.3 (B), SW_NUM-FWD-SLH1.4 (B), SW_NUM6.3 (B), SW_NUM6.4 (B), SW_NUM9.3 (B), SW_NUM9.4 (B), SW_SCRL-LK1.3 (B), SW_SCRL-LK1.4 (B)
- net COL_2: now also SW_1.2 (B), SW_A1.2 (B), SW_ESC1.2 (B), SW_PSE-BK1.2 (B), SW_Q1.2 (B), SW_WIN1.2 (B), SW_Z1.2 (B); no longer SW_1.3 (B), SW_1.4 (B), SW_A1.3 (B), SW_A1.4 (B), SW_ESC1.3 (B), SW_ESC1.4 (B), SW_PSE-BK1.3 (B), SW_PSE-BK1.4 (B), SW_Q1.3 (B), SW_Q1.4 (B), SW_WIN1.3 (B), SW_WIN1.4 (B), SW_Z1.3 (B), SW_Z1.4 (B)
- net COL_3: now also SW_2.2 (B), SW_F1.2 (B), SW_FN1.2 (B), SW_NUM-ASTR1.2 (B), SW_S1.2 (B), SW_W1.2 (B), SW_X1.2 (B); no longer SW_2.3 (B), SW_2.4 (B), SW_F1.3 (B), SW_F1.4 (B), SW_FN1.3 (B), SW_FN1.4 (B), SW_NUM-ASTR1.3 (B), SW_NUM-ASTR1.4 (B), SW_S1.3 (B), SW_S1.4 (B), SW_W1.3 (B), SW_W1.4 (B), SW_X1.3 (B), SW_X1.4 (B)
- net COL_4: now also SW_3.2 (B), SW_C1.2 (B), SW_D1.2 (B), SW_E1.2 (B), SW_F2.2 (B), SW_L-ALT1.2 (B), SW_NUM-MINUS1.2 (B); no longer SW_3.3 (B), SW_3.4 (B), SW_C1.3 (B), SW_C1.4 (B), SW_D1.3 (B), SW_D1.4 (B), SW_E1.3 (B), SW_E1.4 (B), SW_F2.3 (B), SW_F2.4 (B), SW_L-ALT1.3 (B), SW_L-ALT1.4 (B), SW_NUM-MINUS1.3 (B), SW_NUM-MINUS1.4 (B)
- net COL_5: now also SW_4.2 (B), SW_F13.2 (B), SW_F3.2 (B), SW_NUM-PLUS1.2 (B), SW_R1.2 (B), SW_SPACE1.2 (B), SW_V1.2 (B); no longer SW_4.3 (B), SW_4.4 (B), SW_F13.3 (B), SW_F13.4 (B), SW_F3.3 (B), SW_F3.4 (B), SW_NUM-PLUS1.3 (B), SW_NUM-PLUS1.4 (B), SW_R1.3 (B), SW_R1.4 (B), SW_SPACE1.3 (B), SW_SPACE1.4 (B), SW_V1.3 (B), SW_V1.4 (B)
- net COL_6: now also SW_5.2 (B), SW_ALT1.2 (B), SW_B1.2 (B), SW_F4.2 (B), SW_G1.2 (B), SW_PG-UP1.2 (B), SW_T1.2 (B); no longer SW_5.3 (B), SW_5.4 (B), SW_ALT1.3 (B), SW_ALT1.4 (B), SW_B1.3 (B), SW_B1.4 (B), SW_F4.3 (B), SW_F4.4 (B), SW_G1.3 (B), SW_G1.4 (B), SW_PG-UP1.3 (B), SW_PG-UP1.4 (B), SW_T1.3 (B), SW_T1.4 (B)
- net COL_7: now also SW_6.2 (B), SW_F5.2 (B), SW_H1.2 (B), SW_MENU1.2 (B), SW_N1.2 (B), SW_PG-DN1.2 (B), SW_Y1.2 (B); no longer SW_6.3 (B), SW_6.4 (B), SW_F5.3 (B), SW_F5.4 (B), SW_H1.3 (B), SW_H1.4 (B), SW_MENU1.3 (B), SW_MENU1.4 (B), SW_N1.3 (B), SW_N1.4 (B), SW_PG-DN1.3 (B), SW_PG-DN1.4 (B), SW_Y1.3 (B), SW_Y1.4 (B)
- net COL_8: now also SW_7.2 (B), SW_F6.2 (B), SW_J1.2 (B), SW_M1.2 (B), SW_NUM-LK1.2 (B), SW_R-CTRL1.2 (B), SW_U1.2 (B); no longer SW_7.3 (B), SW_7.4 (B), SW_F6.3 (B), SW_F6.4 (B), SW_J1.3 (B), SW_J1.4 (B), SW_M1.3 (B), SW_M1.4 (B), SW_NUM-LK1.3 (B), SW_NUM-LK1.4 (B), SW_R-CTRL1.3 (B), SW_R-CTRL1.4 (B), SW_U1.3 (B), SW_U1.4 (B)
- net COL_9: now also SW_8.2 (B), SW_F7.2 (B), SW_I1.2 (B), SW_K1.2 (B), SW_NUM0.2 (B), SW_OPN-BRC1.2 (B); no longer SW_8.3 (B), SW_8.4 (B), SW_F7.3 (B), SW_F7.4 (B), SW_I1.3 (B), SW_I1.4 (B), SW_K1.3 (B), SW_K1.4 (B), SW_NUM0.3 (B), SW_NUM0.4 (B), SW_OPN-BRC1.3 (B), SW_OPN-BRC1.4 (B)
- net GNDREF: no longer SW_RESET1.2 (A)
- net RESET: now also R9.1, SW_RESET1.2 (B), U1.13 (~{RESET})
- net at D73.2 (A), SW_DELETE1.1 (A): no longer SW_DELETE1.2 (A)
- net at D40.2 (A), SW_Y1.1 (A): no longer SW_Y1.2 (A)
- net at D34.2 (A), SW_G1.1 (A): no longer SW_G1.2 (A)
- net at D17.2 (A), SW_X1.1 (A): no longer SW_X1.2 (A)
- net at D28.2 (A), SW_F13.1 (A): no longer SW_F13.2 (A)
- net at D92.2 (A), SW_SCRL-LK1.1 (A): no longer SW_SCRL-LK1.2 (A)
- net at D67.2 (A), SW_END1.1 (A): no longer SW_END1.2 (A)
- net at D103.2 (A), SW_PG-DN1.1 (A): no longer SW_PG-DN1.2 (A)
- net at D101.2 (A), SW_NUM-PLUS1.1 (A): no longer SW_NUM-PLUS1.2 (A)
- net at D26.2 (A), SW_4.1 (A): no longer SW_4.2 (A)
- net at D1.2 (A), SW_INSERT1.1 (A): no longer SW_INSERT1.2 (A)
- net at D69.2 (A), SW_OPN-BRC2.1 (A): no longer SW_OPN-BRC2.2 (A)
- net at D23.2 (A), SW_C1.1 (A): no longer SW_C1.2 (A)
- net at D87.2 (A), SW_NUM7.1 (A): no longer SW_NUM7.2 (A)
- net at D18.2 (A), SW_FN1.1 (A): no longer SW_FN1.2 (A)
- net at D38.2 (A), SW_F5.1 (A): no longer SW_F5.2 (A)
- net at D33.2 (A), SW_T1.1 (A): no longer SW_T1.2 (A)
- net at D58.2 (A), SW_L1.1 (A): no longer SW_L1.2 (A)
- net at D35.2 (A), SW_B1.1 (A): no longer SW_B1.2 (A)
- net at D63.2 (A), SW_P1.1 (A): no longer SW_P1.2 (A)
- net at D78.2 (A), SW_NUM3.1 (A): no longer SW_NUM3.2 (A)
- net at D48.2 (A), SW_R-CTRL1.1 (A): no longer SW_R-CTRL1.2 (A)
- net at D83.2 (A), SW_DOWN1.1 (A): no longer SW_DOWN1.2 (A)
- net at D2.2 (A), SW_TILDA1.1 (A): no longer SW_TILDA1.2 (A)
- net at D22.2 (A), SW_D1.1 (A): no longer SW_D1.2 (A)
- net at D11.2 (A), SW_Z1.1 (A): no longer SW_Z1.2 (A)
- net at D24.2 (A), SW_L-ALT1.1 (A): no longer SW_L-ALT1.2 (A)
- net at D8.2 (A), SW_1.1 (A): no longer SW_1.2 (A)
- net at D55.2 (A), SW_F8.1 (A): no longer SW_F8.2 (A)
- net at D100.2 (A), SW_NUM-MINUS1.1 (A): no longer SW_NUM-MINUS1.2 (A)
- net at D71.2 (A), SW_R-SHFT1.1 (A): no longer SW_R-SHFT1.2 (A)
- net at D53.2 (A), SW_OPN-BRC1.1 (A): no longer SW_OPN-BRC1.2 (A)
- net at D41.2 (A), SW_H1.1 (A): no longer SW_H1.2 (A)
- net at D89.2 (A), SW_RIGHT1.1 (A): no longer SW_RIGHT1.2 (A)
- net at D64.2 (A), SW_COLON1.1 (A): no longer SW_COLON1.2 (A)
- net at D49.2 (A), SW_F7.1 (A): no longer SW_F7.2 (A)
- net at D82.2 (A), SW_UP1.1 (A): no longer SW_UP1.2 (A)
- net at D6.2 (A), SW_L-CTRL1.1 (A): no longer SW_L-CTRL1.2 (A)
- net at D31.2 (A), SW_F4.1 (A): no longer SW_F4.2 (A)
- net at D98.2 (A), SW_PSE-BK1.1 (A): no longer SW_PSE-BK1.2 (A)
- net at D59.2 (A), SW_CLS-BRC1.1 (A): no longer SW_CLS-BRC1.2 (A)
- net at D44.2 (A), SW_7.1 (A): no longer SW_7.2 (A)
- net at D66.2 (A), SW_NUM1.1 (A): no longer SW_NUM1.2 (A)
- net at D43.2 (A), SW_F6.1 (A): no longer SW_F6.2 (A)
- net at D77.2 (A), SW_LEFT1.1 (A): no longer SW_LEFT1.2 (A)
- net at D79.2 (A), SW_F9.1 (A): no longer SW_F9.2 (A)
- net at D70.2 (A), SW_QUOTE1.1 (A): no longer SW_QUOTE1.2 (A)
- net at D91.2 (A), SW_F11.1 (A): no longer SW_F11.2 (A)
- net at D86.2 (A), SW_PRT-SC1.1 (A): no longer SW_PRT-SC1.2 (A)
- net at D88.2 (A), SW_NUM8.1 (A): no longer SW_NUM8.2 (A)
- net at D60.2 (A), SW_NUM-DEL1.1 (A): no longer SW_NUM-DEL1.2 (A)
- net at D72.2 (A), SW_NUM2.1 (A): no longer SW_NUM2.2 (A)
- net at D51.2 (A), SW_I1.1 (A): no longer SW_I1.2 (A)
- net at D47.2 (A), SW_M1.1 (A): no longer SW_M1.2 (A)
- net at D14.2 (A), SW_2.1 (A): no longer SW_2.2 (A)
- net at D19.2 (A), SW_F2.1 (A): no longer SW_F2.2 (A)
- net at D56.2 (A), SW_9.1 (A): no longer SW_9.2 (A)
- net at D93.2 (A), SW_NUM-FWD-SLH1.1 (A): no longer SW_NUM-FWD-SLH1.2 (A)
- net at D21.2 (A), SW_E1.1 (A): no longer SW_E1.2 (A)
- net at D13.2 (A), SW_F1.1 (A): no longer SW_F1.2 (A)
- net at D68.2 (A), SW_DASH1.1 (A): no longer SW_DASH1.2 (A)
- net at D104.2 (A), SW_NUM-LK1.1 (A): no longer SW_NUM-LK1.2 (A)
- net at D52.2 (A), SW_K1.1 (A): no longer SW_K1.2 (A)
- net at D97.2 (A), SW_F12.1 (A): no longer SW_F12.2 (A)
- net at D39.2 (A), SW_6.1 (A): no longer SW_6.2 (A)
- net at D74.2 (A), SW_PLUS1.1 (A): no longer SW_PLUS1.2 (A)
- net at D94.2 (A), SW_NUM9.1 (A): no longer SW_NUM9.2 (A)
- net at D45.2 (A), SW_U1.1 (A): no longer SW_U1.2 (A)
- net at D15.2 (A), SW_W1.1 (A): no longer SW_W1.2 (A)
- net at D102.2 (A), SW_PG-UP1.1 (A): no longer SW_PG-UP1.2 (A)
- net at D80.2 (A), SW_BACKSPACE1.1 (A): no longer SW_BACKSPACE1.2 (A)
- net at D25.2 (A), SW_F3.1 (A): no longer SW_F3.2 (A)
- net at D65.2 (A), SW_QSTN1.1 (A): no longer SW_QSTN1.2 (A)
- net at D81.2 (A), SW_BK-SLH1.1 (A): no longer SW_BK-SLH1.2 (A)
- net at D30.2 (A), SW_SPACE1.1 (A): no longer SW_SPACE1.2 (A)
- net at D99.2 (A), SW_NUM-ASTR1.1 (A): no longer SW_NUM-ASTR1.2 (A)
- net at D7.2 (A), SW_ESC1.1 (A): no longer SW_ESC1.2 (A)
- net at D95.2 (A), SW_NUM6.1 (A): no longer SW_NUM6.2 (A)
- net at D62.2 (A), SW_0.1 (A): no longer SW_0.2 (A)
- net at D27.2 (A), SW_R1.1 (A): no longer SW_R1.2 (A)
- net at D20.2 (A), SW_3.1 (A): no longer SW_3.2 (A)
- net at D90.2 (A), SW_NUM5.1 (A): no longer SW_NUM5.2 (A)
- net at D3.2 (A), SW_TAB1.1 (A): no longer SW_TAB1.2 (A)
- net at D37.2 (A), SW_N1.1 (A): no longer SW_N1.2 (A)
- net at D61.2 (A), SW_HOME1.1 (A): no longer SW_HOME1.2 (A)
- net at D10.2 (A), SW_A1.1 (A): no longer SW_A1.2 (A)
- net at D85.2 (A), SW_F10.1 (A): no longer SW_F10.2 (A)
- net at D4.2 (A), SW_CAPS1.1 (A): no longer SW_CAPS1.2 (A)
- net at D16.2 (A), SW_S1.1 (A): no longer SW_S1.2 (A)
- net at D75.2 (A), SW_CLO-BRC1.1 (A): no longer SW_CLO-BRC1.2 (A)
- net at D42.2 (A), SW_MENU1.1 (A): no longer SW_MENU1.2 (A)
- net at D29.2 (A), SW_V1.1 (A): no longer SW_V1.2 (A)
- net at D76.2 (A), SW_ENT1.1 (A): no longer SW_ENT1.2 (A)
- net at D9.2 (A), SW_Q1.1 (A): no longer SW_Q1.2 (A)
- net at D32.2 (A), SW_5.1 (A): no longer SW_5.2 (A)
- net at D50.2 (A), SW_8.1 (A): no longer SW_8.2 (A)
- net at D96.2 (A), SW_NUM-ENT1.1 (A): no longer SW_NUM-ENT1.2 (A)
- net at D46.2 (A), SW_J1.1 (A): no longer SW_J1.2 (A)
- net at D36.2 (A), SW_ALT1.1 (A): no longer SW_ALT1.2 (A)
- net at D54.2 (A), SW_NUM0.1 (A): no longer SW_NUM0.2 (A)
- net at D12.2 (A), SW_WIN1.1 (A): no longer SW_WIN1.2 (A)
- net at D84.2 (A), SW_NUM4.1 (A): no longer SW_NUM4.2 (A)
- net at D5.2 (A), SW_L-SHFT1.1 (A): no longer SW_L-SHFT1.2 (A)
- net at D57.2 (A), SW_O1.1 (A): no longer SW_O1.2 (A)
- removed net RST: R9.1, SW_RESET1.3 (B), SW_RESET1.4 (B), U1.13 (~{RESET})
