File: kicad_project_files/keych&chong/keych&chong.kicad_sch (KiCad schematic)
At the start: 228 parts, among them J1 USB_C_Receptacle_USB2.0, U1 ATmega32U4-A, Y1 16mhz

Commit message: place keys on pcb
Parts:
- J1: footprint (none) -> Connector_USB:USB_C_Receptacle_HRO_TYPE-C-31-M-12
- R3, R4, R5, R6, R7, R8, R9: footprint (none) -> Resistor_SMD:R_1206_3216Metric_Pad1.30x1.75mm_HandSolder
Changed lines of the file:
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@@
     (stroke (width 0) (type default) (color 0 0 0 0))
   )
-  (wire (pts (xy 373.38 53.34) (xy 378.46 53.34))
-    (stroke (width 0) (type default) (color 0 0 0 0))
-  )
   (wire (pts (xy 238.76 129.54) (xy 238.76 151.13))
     (stroke (width 0) (type default) (color 0 0 0 0))
@@
     (property "Reference" "R3" (id 0) (at 378.46 176.53 90))
     (property "Value" "5.1K" (id 1) (at 378.46 179.07 90))
-    (property "Footprint" "" (id 2) (at 378.46 180.848 90)
+    (property "Footprint" "Resistor_SMD:R_1206_3216Metric_Pad1.30x1.75mm_HandSolder" (id 2) (at 378.46 180.848 90)
       (effects (font (size 1.27 1.27)) hide)
     )
@@
       (effects (font (size 1.27 1.27)) (justify right))
     )
-    (property "Footprint" "" (id 2) (at 372.618 138.43 90)
+    (property "Footprint" "Resistor_SMD:R_1206_3216Metric_Pad1.30x1.75mm_HandSolder" (id 2) (at 372.618 138.43 90)
       (effects (font (size 1.27 1.27)) hide)
     )
@@
     (property "Reference" "R6" (id 0) (at 378.46 190.5 90))
     (property "Value" "22ohm" (id 1) (at 378.46 187.96 90))
-    (property "Footprint" "" (id 2) (at 378.46 187.96 0)
+    (property "Footprint" "Resistor_SMD:R_1206_3216Metric_Pad1.30x1.75mm_HandSolder" (id 2) (at 378.46 187.96 0)
       (effects (font (size 1.27 1.27)) hide)
     )
@@
       (effects (font (size 1.27 1.27)) (justify left))
     )
-    (property "Footprint" "" (id 2) (at 346.202 219.71 90)
+    (property "Footprint" "Resistor_SMD:R_1206_3216Metric_Pad1.30x1.75mm_HandSolder" (id 2) (at 346.202 219.71 90)
       (effects (font (size 1.27 1.27)) hide)
     )
@@
     (property "Reference" "R8" (id 0) (at 252.73 237.49 90))
     (property "Value" "10k" (id 1) (at 252.73 240.03 90))
-    (property "Footprint" "" (id 2) (at 252.73 241.808 90)
+    (property "Footprint" "Resistor_SMD:R_1206_3216Metric_Pad1.30x1.75mm_HandSolder" (id 2) (at 252.73 241.808 90)
       (effects (font (size 1.27 1.27)) hide)
     )
@@
     (property "Reference" "R4" (id 0) (at 378.46 184.15 90))
     (property "Value" "5.1k" (id 1) (at 378.46 181.61 90))
-    (property "Footprint" "" (id 2) (at 378.46 183.388 90)
+    (property "Footprint" "Resistor_SMD:R_1206_3216Metric_Pad1.30x1.75mm_HandSolder" (id 2) (at 378.46 183.388 90)
       (effects (font (size 1.27 1.27)) hide)
     )
@@
     (property "Reference" "R7" (id 0) (at 378.46 195.58 90))
     (property "Value" "22ohm" (id 1) (at 378.46 193.04 90))
-    (property "Footprint" "" (id 2) (at 378.46 193.04 0)
+    (property "Footprint" "Resistor_SMD:R_1206_3216Metric_Pad1.30x1.75mm_HandSolder" (id 2) (at 378.46 193.04 0)
       (effects (font (size 1.27 1.27)) hide)
     )
@@
     (property "Reference" "J1" (id 0) (at 355.6 166.37 0))
     (property "Value" "USB_C_Receptacle_USB2.0" (id 1) (at 355.6 168.91 0))
-    (property "Footprint" "" (id 2) (at 359.41 189.23 0)
+    (property "Footprint" "Connector_USB:USB_C_Receptacle_HRO_TYPE-C-31-M-12" (id 2) (at 359.41 189.23 0)
       (effects (font (size 1.27 1.27)) hide)
     )
@@
     )
     (path "/feeb1353-42f7-48c2-a822-76be09b16b85"
-      (reference "J1") (unit 1) (value "USB_C_Receptacle_USB2.0") (footprint "")
+      (reference "J1") (unit 1) (value "USB_C_Receptacle_USB2.0") (footprint "Connector_USB:USB_C_Receptacle_HRO_TYPE-C-31-M-12")
     )
     (path "/6eb6978a-b62b-4e04-a66d-dad3ed2eccc1"
@@
     )
     (path "/0a5b922a-c7a7-4407-a015-24de7e4c2887"
-      (reference "R3") (unit 1) (value "5.1K") (footprint "")
+      (reference "R3") (unit 1) (value "5.1K") (footprint "Resistor_SMD:R_1206_3216Metric_Pad1.30x1.75mm_HandSolder")
     )
     (path "/ad6d76a0-fc1a-4c80-96a8-0add704fe474"
-      (reference "R4") (unit 1) (value "5.1k") (footprint "")
+      (reference "R4") (unit 1) (value "5.1k") (footprint "Resistor_SMD:R_1206_3216Metric_Pad1.30x1.75mm_HandSolder")
     )
     (path "/2f564b3f-c9b1-40cc-95b3-e5c0a79e748b"
-      (reference "R5") (unit 1) (value "1M") (footprint "")
+      (reference "R5") (unit 1) (value "1M") (footprint "Resistor_SMD:R_1206_3216Metric_Pad1.30x1.75mm_HandSolder")
     )
     (path "/2bc894ed-b163-4717-833e-b598cfa1d86e"
-      (reference "R6") (unit 1) (value "22ohm") (footprint "")
+      (reference "R6") (unit 1) (value "22ohm") (footprint "Resistor_SMD:R_1206_3216Metric_Pad1.30x1.75mm_HandSolder")
     )
     (path "/b19e45ae-9b9d-4b8a-9939-5787fb3aaee4"
-      (reference "R7") (unit 1) (value "22ohm") (footprint "")
+      (reference "R7") (unit 1) (value "22ohm") (footprint "Resistor_SMD:R_1206_3216Metric_Pad1.30x1.75mm_HandSolder")
     )
     (path "/4b36f467-2d4e-43cf-9ce6-750edb207425"
-      (reference "R8") (unit 1) (value "10k") (footprint "")
+      (reference "R8") (unit 1) (value "10k") (footprint "Resistor_SMD:R_1206_3216Metric_Pad1.30x1.75mm_HandSolder")
     )
     (path "/1a8a54cb-a7d6-4c4a-a829-7f3a5efc51aa"
-      (reference "R9") (unit 1) (value "10k") (footprint "")
+      (reference "R9") (unit 1) (value "10k") (footprint "Resistor_SMD:R_1206_3216Metric_Pad1.30x1.75mm_HandSolder")
     )
     (path "/74e04d55-3406-412a-8d4d-73659f0bd63a"

Commit message: place diodes
Parts:
- SW_RESET1: footprint Button_Switch_Keyboard:SW_Cherry_MX_1.00u_Plate -> Button - Alternate:SW_4-1437565-0
Changed lines of the file:
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@@
     (property "Reference" "SW_RESET1" (id 0) (at 361.95 137.16 0))
     (property "Value" "SW_SPST" (id 1) (at 361.95 139.7 0))
-    (property "Footprint" "Button_Switch_Keyboard:SW_Cherry_MX_1.00u_Plate" (id 2) (at 361.95 144.78 0)
+    (property "Footprint" "Button - Alternate:SW_4-1437565-0" (id 2) (at 361.95 144.78 0)
       (effects (font (size 1.27 1.27)) hide)
     )
@@
     )
     (path "/f73d5f45-bf04-4553-a792-1e4a94053fa4"
-      (reference "SW_RESET1") (unit 1) (value "SW_SPST") (footprint "Button_Switch_Keyboard:SW_Cherry_MX_1.00u_Plate")
+      (reference "SW_RESET1") (unit 1) (value "SW_SPST") (footprint "Button - Alternate:SW_4-1437565-0")
     )
     (path "/6b43eec3-dc09-4354-a1be-2eb407f4bef4"
