File: kicad_project_files/keych&chong/keych&chong.kicad_pcb (KiCad board)
At the start: 2 copper layers, 228 parts, among them J1 USB_C_Receptacle_USB2.0, U1 ATmega32U4-A, Y1 16mhz

Commit message: place diodes
Parts:
- SW_RESET1: footprint Button_Switch_Keyboard:SW_Cherry_MX_1.00u_Plate -> Button - Alternate:SW_4-1437565-0
- moved D1 745.1 mm to (47.6, 32.2)
- moved D2 732.2 mm to (45.2, 60.9)
- moved D18 723.2 mm to (71.2, 137.5)
- moved D8 706.8 mm to (65.0, 60.4)
- moved D24 699.7 mm to (119.3, 136.8)
- moved D5 697.5 mm to (57.9, 117.5)
- moved D13 684.8 mm to (103.2, 32.4)
- moved D14 683.6 mm to (84.9, 60.9)
- moved D9 673.7 mm to (74.7, 80.0)
- moved D29 672.7 mm to (146.4, 118.4)
- moved D34 671.7 mm to (155.3, 99.1)
- moved D26 670.5 mm to (121.8, 61.2)
- moved D10 661.8 mm to (79.8, 99.1)
- moved D33 646.3 mm to (150.6, 79.8)
- moved D11 645.2 mm to (90.2, 117.9)
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Connections:
- SW_0 pad 1: (no net) -> Net-(D62-Pad2)
- SW_0 pad 2: (no net) -> COL_11
- SW_2 pad 1: (no net) -> Net-(D14-Pad2)
- SW_2 pad 2: (no net) -> COL_3
- SW_5 pad 1: (no net) -> Net-(D32-Pad2)
- SW_5 pad 2: (no net) -> COL_6
- SW_6 pad 1: (no net) -> Net-(D39-Pad2)
- SW_6 pad 2: (no net) -> COL_7
- SW_7 pad 1: (no net) -> Net-(D44-Pad2)
- SW_7 pad 2: (no net) -> COL_8
- SW_8 pad 1: (no net) -> Net-(D50-Pad2)
- SW_8 pad 2: (no net) -> COL_9
- SW_A1 pad 1: (no net) -> Net-(D10-Pad2)
- SW_A1 pad 2: (no net) -> COL_2
- SW_ALT1 pad 1: (no net) -> Net-(D36-Pad2)
- SW_ALT1 pad 2: (no net) -> COL_6
- SW_ARR_BRK_C1 pad 1: (no net) -> Net-(D59-Pad2)
- SW_ARR_BRK_C1 pad 2: (no net) -> COL_10
- SW_ARR_BRK_O1 pad 1: (no net) -> Net-(D53-Pad2)
- SW_ARR_BRK_O1 pad 2: (no net) -> COL_9
- SW_B1 pad 1: (no net) -> Net-(D35-Pad2)
- SW_B1 pad 2: (no net) -> COL_6
- SW_C1 pad 1: (no net) -> Net-(D23-Pad2)
- SW_C1 pad 2: (no net) -> COL_4
- SW_CAPS1 pad 1: (no net) -> Net-(D4-Pad2)
- SW_CAPS1 pad 2: (no net) -> COL_1
- SW_D1 pad 1: (no net) -> Net-(D22-Pad2)
- SW_D1 pad 2: (no net) -> COL_4
- SW_E1 pad 1: (no net) -> Net-(D21-Pad2)
- SW_E1 pad 2: (no net) -> COL_4
- SW_END1 pad 1: (no net) -> Net-(D92-Pad2)
- SW_END1 pad 2: (no net) -> COL_16
- SW_ENT1 pad 1: (no net) -> Net-(D76-Pad2)
- SW_ENT1 pad 2: (no net) -> COL_13
- SW_ESC1 pad 1: (no net) -> Net-(D1-Pad2)
- SW_ESC1 pad 2: (no net) -> COL_1
- SW_F10 pad 1: (no net) -> Net-(D61-Pad2)
- SW_F10 pad 2: (no net) -> COL_11
- SW_F11 pad 1: (no net) -> Net-(D67-Pad2)
- SW_F11 pad 2: (no net) -> COL_12
- SW_F13 pad 1: (no net) -> Net-(D28-Pad2)
- SW_F13 pad 2: (no net) -> COL_5
- SW_F3 pad 1: (no net) -> Net-(D19-Pad2)
- SW_F3 pad 2: (no net) -> COL_4
- SW_F4 pad 1: (no net) -> Net-(D25-Pad2)
- SW_F4 pad 2: (no net) -> COL_5
- SW_F7 pad 1: (no net) -> Net-(D43-Pad2)
- SW_F7 pad 2: (no net) -> COL_8
- SW_F8 pad 1: (no net) -> Net-(D49-Pad2)
- SW_F8 pad 2: (no net) -> COL_9
- SW_FN1 pad 1: (no net) -> Net-(D18-Pad2)
- SW_FN1 pad 2: (no net) -> COL_3
- SW_G1 pad 1: (no net) -> Net-(D34-Pad2)
- SW_G1 pad 2: (no net) -> COL_6
- SW_H1 pad 1: (no net) -> Net-(D41-Pad2)
- SW_H1 pad 2: (no net) -> COL_7
- SW_HOME1 pad 1: (no net) -> Net-(D86-Pad2)
- SW_HOME1 pad 2: (no net) -> COL_15
- SW_I1 pad 1: (no net) -> Net-(D51-Pad2)
- SW_I1 pad 2: (no net) -> COL_9
- SW_INSERT1 pad 1: (no net) -> Net-(D79-Pad2)
- SW_INSERT1 pad 2: (no net) -> COL_14
- SW_J1 pad 1: (no net) -> Net-(D46-Pad2)
- SW_J1 pad 2: (no net) -> COL_8
- SW_K1 pad 1: (no net) -> Net-(D52-Pad2)
- SW_K1 pad 2: (no net) -> COL_9
- SW_L-CTRL1 pad 1: (no net) -> Net-(D6-Pad2)
- SW_L-CTRL1 pad 2: (no net) -> COL_1
- SW_L1 pad 1: (no net) -> Net-(D58-Pad2)
- SW_L1 pad 2: (no net) -> COL_10
- SW_LEFT1 pad 1: (no net) -> Net-(D54-Pad2)
- SW_LEFT1 pad 2: (no net) -> COL_9
- SW_M1 pad 1: (no net) -> Net-(D47-Pad2)
- SW_M1 pad 2: (no net) -> COL_8
- SW_MENU1 pad 1: (no net) -> Net-(D42-Pad2)
- SW_MENU1 pad 2: (no net) -> COL_7
- SW_N1 pad 1: (no net) -> Net-(D37-Pad2)
- SW_N1 pad 2: (no net) -> COL_7
- SW_NUM-ASTR1 pad 1: (no net) -> Net-(D99-Pad2)
- SW_NUM-ASTR1 pad 2: (no net) -> COL_17
- SW_NUM-DEL1 pad 1: (no net) -> Net-(D78-Pad2)
- SW_NUM-DEL1 pad 2: (no net) -> COL_13
- SW_NUM-ENT1 pad 1: (no net) -> Net-(D102-Pad2)
- SW_NUM-ENT1 pad 2: (no net) -> COL_17
- SW_NUM-FWD-SLH1 pad 1: (no net) -> Net-(D93-Pad2)
- SW_NUM-FWD-SLH1 pad 2: (no net) -> COL_16
- SW_NUM-LK1 pad 1: (no net) -> Net-(D87-Pad2)
- SW_NUM-LK1 pad 2: (no net) -> COL_15
- SW_NUM-MINUS1 pad 1: (no net) -> Net-(D97-Pad2)
- SW_NUM-MINUS1 pad 2: (no net) -> COL_17
- SW_NUM-PLUS1 pad 1: (no net) -> Net-(D98-Pad2)
- SW_NUM-PLUS1 pad 2: (no net) -> COL_17
- SW_NUM2 pad 1: (no net) -> Net-(D90-Pad2)
- SW_NUM2 pad 2: (no net) -> COL_15
- SW_O1 pad 1: (no net) -> Net-(D57-Pad2)
- SW_O1 pad 2: (no net) -> COL_10
- SW_OPN-BRC1 pad 1: (no net) -> Net-(D69-Pad2)
- SW_OPN-BRC1 pad 2: (no net) -> COL_12
- SW_P1 pad 1: (no net) -> Net-(D63-Pad2)
- SW_P1 pad 2: (no net) -> COL_11
- SW_PG-UP1 pad 1: (no net) -> Net-(D82-Pad2)
- SW_PG-UP1 pad 2: (no net) -> COL_14
- SW_PRT-SC1 pad 1: (no net) -> Net-(D85-Pad2)
- SW_PRT-SC1 pad 2: (no net) -> COL_15
- SW_Q1 pad 1: (no net) -> Net-(D9-Pad2)
- SW_Q1 pad 2: (no net) -> COL_2
- SW_QSTN1 pad 1: (no net) -> Net-(D65-Pad2)
- SW_QSTN1 pad 2: (no net) -> COL_11
- SW_QUOTE1 pad 1: (no net) -> Net-(D70-Pad2)
- SW_QUOTE1 pad 2: (no net) -> COL_12
- SW_R-CTRL1 pad 1: (no net) -> Net-(D48-Pad2)
- SW_R-CTRL1 pad 2: (no net) -> COL_8
- SW_R-SHFT1 pad 1: (no net) -> Net-(D71-Pad2)
- SW_R-SHFT1 pad 2: (no net) -> COL_12
- SW_R1 pad 1: (no net) -> Net-(D27-Pad2)
- SW_R1 pad 2: (no net) -> COL_5
- SW_T1 pad 1: (no net) -> Net-(D33-Pad2)
- SW_T1 pad 2: (no net) -> COL_6
- SW_U1 pad 1: (no net) -> Net-(D45-Pad2)
- SW_U1 pad 2: (no net) -> COL_8
- SW_UP1 pad 1: (no net) -> Net-(D77-Pad2)
- SW_UP1 pad 2: (no net) -> COL_13
- SW_V1 pad 1: (no net) -> Net-(D29-Pad2)
- SW_V1 pad 2: (no net) -> COL_5
- SW_W1 pad 1: (no net) -> Net-(D15-Pad2)
- SW_W1 pad 2: (no net) -> COL_3
- SW_WIN1 pad 1: (no net) -> Net-(D12-Pad2)
- SW_WIN1 pad 2: (no net) -> COL_2
- SW_X1 pad 1: (no net) -> Net-(D17-Pad2)
- SW_X1 pad 2: (no net) -> COL_3
- SW_Y1 pad 1: (no net) -> Net-(D40-Pad2)
- SW_Y1 pad 2: (no net) -> COL_7
- SW_Z1 pad 1: (no net) -> Net-(D11-Pad2)
- SW_Z1 pad 2: (no net) -> COL_2

Commit message: align diodes
Parts:
- moved R9 206.9 mm to (463.5, 42.2), turned to 90 degrees
- moved R7 142.5 mm to (254.5, 20.3), turned to -90 degrees
- moved R8 33.5 mm to (406.4, 38.1), turned to 45 degrees
- moved C1 25.9 mm to (388.1, 49.3), turned to 135 degrees
- moved C2 25.1 mm to (382.4, 43.5), turned to -45 degrees
- moved R6 18.8 mm to (237.9, 20.3), turned to -90 degrees
- moved Y1 18.5 mm to (386.7, 41.6), turned to -45 degrees
- moved R4 18.1 mm to (235.5, 20.3), turned to 90 degrees
- moved C8 18.0 mm to (399.9, 44.5), turned to -135 degrees
- moved R3 16.9 mm to (252.1, 20.3), turned to 90 degrees
- moved C5 15.8 mm to (404.3, 30.7), turned to 135 degrees
- moved C4 15.3 mm to (406.2, 28.6), turned to 135 degrees
- moved R5 14.5 mm to (256.9, 20.3), turned to 90 degrees
- moved C3 12.5 mm to (389.1, 29.1), turned to 45 degrees
- moved D66 8.71 mm to (371.1, 142.4), turned to 180 degrees
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