File: kicad_project_files/atmega32u4-prototype/atmega32u4-prototype.kicad_sch (KiCad schematic)
At the start: 40 parts, among them J1 Conn_02x03_Odd_Even, J2 USB_C_Receptacle_USB2.0, SW1 SW_Push, SW2 SW_Push, SW3 SW_Push, SW4 SW_Push, SW5 SW_Push, SW6 SW_Push, SW7 SW_Push, SW8 SW_Push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

Commit message: assign footprints
Parts:
- C1, C2, C3, C4: footprint (none) -> Capacitor_THT:C_Rect_L7.0mm_W2.0mm_P5.00mm
- C5: footprint (none) -> Capacitor_THT:CP_Radial_D6.3mm_P2.50mm
- C6, C9: footprint (none) -> Capacitor_THT:CP_Radial_D4.0mm_P1.50mm
- C7, C8: footprint (none) -> Capacitor_THT:C_Disc_D3.0mm_W1.6mm_P2.50mm
- D_CAPS1: footprint (none) -> LED_THT:LED_D3.0mm
- J1: footprint (none) -> Connector_PinHeader_2.54mm:PinHeader_2x03_P2.54mm_Vertical
- J2: footprint (none) -> Connector_USB:USB_C_Receptacle_HRO_TYPE-C-31-M-12
- R1, R2, R3, R4, R5, R6, R7: footprint (none) -> Resistor_THT:R_Axial_DIN0207_L6.3mm_D2.5mm_P7.62mm_Horizontal
- SW1, SW2, SW3, SW4, SW5, SW6, SW7, SW8, SW_CAPS1, SW_RESET1: footprint (none) -> Button - Alternate:SW_4-1437565-0
- Y1: footprint (none) -> Crystal:Crystal_HC49-4H_Vertical
